Commit message: Ajout perception YOLO, tests de repetabilite et integration trac_ik
- Nouveau package perception/ : detection d'objets (camera + robot),
  homographie camera-bras, landmarks, launch files de vision
- Package yolo/ : scripts d'entrainement et de detection YOLO
- mon_controleur : nouveaux noeuds (test_repetabilite, workspace_scene,
  go_homepick, pick_place cartesien/optim, robot_dance) et launch files
- Mise a jour pick_place_ia, securite, setup.py
- Integration de la bibliotheque trac_ik (solveur cinematique)
- Mise a jour URDF (cameras, gripper Schunk) et config MoveIt
- Rapport de repetabilite
- Nettoyage : suppression des scripts obsoletes et des fichiers .pyc,
  .gitignore enrichi (cache Python, modeles, outils)

Co-Authored-By: Claude Opus 4.7 <noreply@anthropic.com>

File: src/ros2-igus-rebel/igus_rebel_description_ros2/urdf/cameras/cameras.urdf.xacro (robot description, xacro)
@@ -2,6 +2,7 @@
 <robot xmlns:xacro="http://www.ros.org/wiki/xacro" name="igus_rebel">
     <xacro:macro name="cameras" params="camera load_gazebo">
-        <!-- virtual frames for gazebo -->
-        <xacro:if value="${load_gazebo}">
+        <!-- virtual frames for gazebo — uniquement si une caméra est montée sur le bras -->
+        <!-- camera=none + load_gazebo=true → pas de camera_link → URDF cassé sans cette garde -->
+        <xacro:if value="${load_gazebo and camera != 'none'}">
             <xacro:include
                 filename="$(find igus_rebel_description_ros2)/urdf/cameras/virtual_camera_frames.xacro" />

File: src/ros2-igus-rebel/igus_rebel_description_ros2/urdf/end_effectors/schunk_egp25.urdf.xacro (robot description, xacro)
@@ -20,5 +20,5 @@
         <origin xyz="0 -0.0375 0.015" rpy="0 0 -1.5708"/>
         <geometry>
-          <mesh filename="package://igus_rebel_description_ros2/meshes/end_effectors/effecteur_simplifie.stl"
+          <mesh filename="file://$(find igus_rebel_description_ros2)/meshes/end_effectors/effecteur_simplifie.stl"
                 scale="0.001 0.001 0.001"/>
         </geometry>
@@ -51,4 +51,10 @@
     </joint>
     <link name="gripper_tip_link"/>
+    <!-- Gazebo : couleur de la pince (bleue) + friction -->
+    <gazebo reference="effecteur_simplifie_link">
+      <material>Gazebo/Blue</material>
+      <mu1>0.8</mu1>
+      <mu2>0.8</mu2>
+    </gazebo>
   </xacro:macro>
 </robot>

File: src/ros2-igus-rebel/igus_rebel_description_ros2/urdf/igus_rebel/igus_rebel.control.xacro (robot description, xacro)
@@ -26,5 +26,5 @@
 				params="name position_min=0 position_max=0 cri_joint_offset=0">
 				<joint name="${name}">
-					<!-- Position control can be optionally deployed -->
+						<!-- Position control can be optionally deployed -->
 					<!--<command_interface
 					name="position">

File: src/ros2-igus-rebel/igus_rebel_description_ros2/urdf/igus_rebel/igus_rebel.description.xacro (robot description, xacro)
@@ -19,6 +19,5 @@
 				<geometry>
 					<mesh
-						filename="file://$(find igus_rebel_description_ros2)/meshes/igus_rebel_mod/Joint0.stl"
-						scale="0.0001 0.0001 0.0001" />
+						filename="file://$(find igus_rebel_description_ros2)/meshes/igus_rebel/Joint0.dae" />
 				</geometry>
 			</collision>
@@ -48,6 +47,5 @@
 				<geometry>
 					<mesh
-						filename="file://$(find igus_rebel_description_ros2)/meshes/igus_rebel_mod/Joint1.stl"
-						scale="0.0001 0.0001 0.0001" />
+						filename="file://$(find igus_rebel_description_ros2)/meshes/igus_rebel/Joint1.dae" />
 				</geometry>
 				<origin rpy="0 0 0" xyz="0 0 0" />
@@ -78,6 +76,5 @@
 				<geometry>
 					<mesh
-						filename="file://$(find igus_rebel_description_ros2)/meshes/igus_rebel_mod/Joint2.stl"
-						scale="0.0001 0.0001 0.0001" />
+						filename="file://$(find igus_rebel_description_ros2)/meshes/igus_rebel/Joint2.dae" />
 				</geometry>
 				<origin rpy="0 0 0" xyz="0 0 0" />
@@ -108,6 +105,5 @@
 				<geometry>
 					<mesh
-						filename="file://$(find igus_rebel_description_ros2)/meshes/igus_rebel_mod/Joint3.stl"
-						scale="0.0001 0.0001 0.0001" />
+						filename="file://$(find igus_rebel_description_ros2)/meshes/igus_rebel/Joint3.dae" />
 				</geometry>
 				<origin rpy="0 0 0" xyz="0 0 0" />
@@ -138,6 +134,5 @@
 				<geometry>
 					<mesh
-						filename="file://$(find igus_rebel_description_ros2)/meshes/igus_rebel_mod/Joint4.stl"
-						scale="0.0001 0.0001 0.0001" />
+						filename="file://$(find igus_rebel_description_ros2)/meshes/igus_rebel/Joint4.dae" />
 				</geometry>
 				<origin rpy="0 0 0" xyz="0 0 0" />
@@ -168,6 +163,5 @@
 				<geometry>
 					<mesh
-						filename="file://$(find igus_rebel_description_ros2)/meshes/igus_rebel_mod/Joint5.stl"
-						scale="0.0001 0.0001 0.0001" />
+						filename="file://$(find igus_rebel_description_ros2)/meshes/igus_rebel/Joint5.dae" />
 				</geometry>
 				<origin rpy="0 0 0" xyz="0 0 0" />
@@ -198,6 +192,5 @@
 				<geometry>
 					<mesh
-						filename="file://$(find igus_rebel_description_ros2)/meshes/igus_rebel_mod/Joint6.stl"
-						scale="0.0001 0.0001 0.0001" />
+						filename="file://$(find igus_rebel_description_ros2)/meshes/igus_rebel/Joint6.dae" />
 				</geometry>
 				<origin rpy="0 0 0" xyz="0.0 0 0" />

File: src/ros2-igus-rebel/igus_rebel_description_ros2/urdf/igus_rebel/igus_rebel.urdf.xacro (robot description, xacro)
@@ -51,5 +51,7 @@
 		</xacro:if>
 		<!-- Chargement conditionnel du Schunk EGP25 (effecteur_simplifie.stl) -->
-		<xacro:if value="${end_effector == 'schunk_egp25'}">
+		<!-- Ne charger que si mount == 'none' pour éviter le conflit de joint parent=flange
+		     avec flange_to_mount défini dans mount_v1/mount_v2 -->
+		<xacro:if value="${end_effector == 'schunk_egp25' and mount == 'none'}">
 			<xacro:include filename="$(find igus_rebel_description_ros2)/urdf/end_effectors/schunk_egp25.urdf.xacro" />
 			<xacro:schunk_gripper />
